File: KiCad/microcontroller.kicad_sch (KiCad schematic)
At the start: 57 parts, among them J4 Debugger, SW1 Reset switch, U7 24LC256

Commit message: lots of suf for pcb diseng
Parts:
- R11, R30, R31, R32, R33, R34, R35, R36, R37, R38, R39, R40, R41, R42, R43, R44, R45, R46, R47, R69, R70, R71, R72: cost per unit (none) -> 0,0010
- R56, R57: cost per unit (none) -> 0,0066
- R64: JLC code (none) -> C17414; Part name (none) -> 0805W8F1002T5E; cost per unit (none) -> 0,0010
Changed lines of the file:
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@@
       (effects (font (size 1.27 1.27)) hide)
     )
-    (property "cost per unit" "" (at 60.96 186.69 0)
+    (property "cost per unit" "0,0010" (at 60.96 186.69 0)
       (effects (font (size 1.27 1.27)) hide)
     )
@@
       (effects (font (size 1.27 1.27)) hide)
     )
-    (property "cost per unit" "" (at 55.88 118.11 0)
+    (property "cost per unit" "0,0010" (at 55.88 118.11 0)
       (effects (font (size 1.27 1.27)) hide)
     )
@@
       (effects (font (size 1.27 1.27)) hide)
     )
-    (property "cost per unit" "" (at 55.88 121.92 0)
+    (property "cost per unit" "0,0010" (at 55.88 121.92 0)
       (effects (font (size 1.27 1.27)) hide)
     )
@@
       (effects (font (size 1.27 1.27)) hide)
     )
-    (property "cost per unit" "" (at 60.96 165.1 0)
+    (property "cost per unit" "0,0010" (at 60.96 165.1 0)
       (effects (font (size 1.27 1.27)) hide)
     )
@@
       (effects (font (size 1.27 1.27)) hide)
     )
-    (property "cost per unit" "" (at 259.08 72.39 0)
+    (property "cost per unit" "0,0010" (at 259.08 72.39 0)
       (effects (font (size 1.27 1.27)) hide)
     )
@@
       (effects (font (size 1.27 1.27)) hide)
     )
-    (property "cost per unit" "" (at 55.88 100.33 0)
+    (property "cost per unit" "0,0010" (at 55.88 100.33 0)
       (effects (font (size 1.27 1.27)) hide)
     )
@@
       (effects (font (size 1.27 1.27)) hide)
     )
-    (property "cost per unit" "" (at 55.88 104.14 0)
+    (property "cost per unit" "0,0010" (at 55.88 104.14 0)
       (effects (font (size 1.27 1.27)) hide)
     )
@@
       (effects (font (size 1.27 1.27)) hide)
     )
-    (property "cost per unit" "" (at 120.65 166.37 0)
+    (property "cost per unit" "0,0066" (at 120.65 166.37 0)
       (effects (font (size 1.27 1.27)) hide)
     )
@@
       (effects (font (size 1.27 1.27)) hide)
     )
-    (property "cost per unit" "" (at 55.88 140.97 0)
+    (property "cost per unit" "0,0010" (at 55.88 140.97 0)
       (effects (font (size 1.27 1.27)) hide)
     )
@@
       (effects (font (size 1.27 1.27)) hide)
     )
-    (property "cost per unit" "" (at 60.96 168.91 0)
+    (property "cost per unit" "0,0010" (at 60.96 168.91 0)
       (effects (font (size 1.27 1.27)) hide)
     )
@@
       (effects (font (size 1.27 1.27)) hide)
     )
-    (property "cost per unit" "" (at 60.96 175.26 0)
+    (property "cost per unit" "0,0010" (at 60.96 175.26 0)
       (effects (font (size 1.27 1.27)) hide)
     )
@@
       (effects (font (size 1.27 1.27)) hide)
     )
-    (property "cost per unit" "" (at 259.08 68.58 0)
+    (property "cost per unit" "0,0010" (at 259.08 68.58 0)
       (effects (font (size 1.27 1.27)) hide)
     )
@@
       (effects (font (size 1.27 1.27)) hide)
     )
-    (property "cost per unit" "" (at 60.96 182.88 0)
+    (property "cost per unit" "0,0010" (at 60.96 182.88 0)
       (effects (font (size 1.27 1.27)) hide)
     )
@@
       (effects (font (size 1.27 1.27)) hide)
     )
-    (property "cost per unit" "" (at 121.158 178.562 0)
+    (property "cost per unit" "0,0066" (at 121.158 178.562 0)
       (effects (font (size 1.27 1.27)) hide)
     )
@@
       (effects (font (size 1.27 1.27)) hide)
     )
-    (property "cost per unit" "" (at 55.88 107.95 0)
+    (property "cost per unit" "0,0010" (at 55.88 107.95 0)
       (effects (font (size 1.27 1.27)) hide)
     )
@@
       (effects (font (size 1.27 1.27)) hide)
     )
-    (property "cost per unit" "" (at 55.753 133.35 0)
+    (property "cost per unit" "0,0010" (at 55.753 133.35 0)
       (effects (font (size 1.27 1.27)) hide)
     )
@@
       (effects (font (size 1.27 1.27)) hide)
     )
-    (property "cost per unit" "" (at 55.88 114.3 0)
+    (property "cost per unit" "0,0010" (at 55.88 114.3 0)
       (effects (font (size 1.27 1.27)) hide)
     )
@@
       (effects (font (size 1.27 1.27)) hide)
     )
-    (property "cost per unit" "" (at 55.88 129.54 0)
+    (property "cost per unit" "0,0010" (at 55.88 129.54 0)
       (effects (font (size 1.27 1.27)) hide)
     )
@@
       (effects (font (size 1.27 1.27)) hide)
     )
-    (property "cost per unit" "" (at 270.51 116.84 0)
+    (property "cost per unit" "0,0010" (at 270.51 116.84 0)
       (effects (font (size 1.27 1.27)) hide)
     )
@@
       (effects (font (size 1.27 1.27)) hide)
     )
-    (property "cost per unit" "" (at 60.96 161.29 0)
+    (property "cost per unit" "0,0010" (at 60.96 161.29 0)
       (effects (font (size 1.27 1.27)) hide)
     )
@@
       (effects (font (size 1.27 1.27)) hide)
     )
-    (property "cost per unit" "" (at 270.51 119.38 0)
+    (property "cost per unit" "0,0010" (at 270.51 119.38 0)
       (effects (font (size 1.27 1.27)) hide)
     )
@@
       (effects (font (size 1.27 1.27)) hide)
     )
-    (property "cost per unit" "" (at 240.03 68.58 0)
+    (property "cost per unit" "0,0010" (at 240.03 68.58 0)
       (effects (font (size 1.27 1.27)) hide)
     )
@@
       (effects (font (size 1.27 1.27)) hide)
     )
-    (property "cost per unit" "" (at 60.96 157.48 0)
+    (property "cost per unit" "0,0010" (at 60.96 157.48 0)
       (effects (font (size 1.27 1.27)) hide)
     )
@@
       (effects (font (size 1.27 1.27)) hide)
     )
-    (property "cost per unit" "" (at 270.51 111.76 0)
+    (property "cost per unit" "0,0010" (at 270.51 111.76 0)
       (effects (font (size 1.27 1.27)) hide)
     )
@@
       (effects (font (size 1.27 1.27)) hide)
     )
-    (property "cost per unit" "" (at 270.51 109.22 0)
+    (property "cost per unit" "0,0010" (at 270.51 109.22 0)
       (effects (font (size 1.27 1.27)) hide)
     )
@@
       (effects (font (size 1.27 1.27)) hide)
     )
-    (property "cost per unit" "" (at 60.96 179.07 0)
+    (property "cost per unit" "0,0010" (at 60.96 179.07 0)
       (effects (font (size 1.27 1.27)) hide)
     )
@@
       (effects (font (size 1.27 1.27)) hide)
     )
-    (property "cost per unit" "" (at 240.03 72.39 0)
+    (property "cost per unit" "0,0010" (at 240.03 72.39 0)
       (effects (font (size 1.27 1.27)) hide)
     )
@@
       (effects (font (size 1.27 1.27)) hide)
     )
-    (property "cost per unit" "" (at 55.88 137.16 0)
+    (property "cost per unit" "0,0010" (at 55.88 137.16 0)
       (effects (font (size 1.27 1.27)) hide)
     )
@@
       (effects (font (size 1.27 1.27)) hide)
     )
-    (property "JLC code" "" (at 201.93 154.94 0)
-      (effects (font (size 1.27 1.27)) hide)
-    )
-    (property "Part name" "" (at 201.93 154.94 0)
-      (effects (font (size 1.27 1.27)) hide)
-    )
-    (property "cost per unit" "" (at 201.93 154.94 0)
-      (effects (font (size 1.27 1.27)) hide)
-    )
+    (property "JLC code" "C17414" (at 201.93 154.94 0)
+      (effects (font (size 1.27 1.27)) hide)
+    )
+    (property "Part name" "0805W8F1002T5E" (at 201.93 154.94 0)
+      (effects (font (size 1.27 1.27)) hide)
+    )
+    (property "cost per unit" "0,0010" (at 201.93 154.94 0)
+      (effects (font (size 1.27 1.27)) hide)
+    )
