File: KiCad/sensors.kicad_sch (KiCad schematic)
At the start: 26 parts, among them Q1 AO3401A, U4 GXHTC3, U5 LTR-303ALS-01

Commit message: footprint added
Parts:
- C1: footprint (none) -> footprint:C0402
- C1: footprint (none) -> footprint:C0402_NEW
- Q1: footprint Package_TO_SOT_SMD:SOT-23 -> footprint:SOT-23_L2.9-W1.3-P1.90-LS2.4-BR
- R11: footprint (none) -> footprint:R0603
- R2: footprint (none) -> footprint:R1206
- RV1: footprint (none) -> footprint:RES-ADJ-TH_RK09K1130AJ3
- TH1: footprint (none) -> footprint:R0402
- TP10: value TestPoint -> Light SCL; footprint (none) -> TestPoint:TestPoint_Loop_D2.54mm_Drill1.5mm_Beaded
- TP11: value TestPoint -> Light Interrupt; footprint (none) -> TestPoint:TestPoint_Loop_D2.54mm_Drill1.5mm_Beaded
- TP12: value TestPoint -> TempHum SDA; footprint (none) -> TestPoint:TestPoint_Loop_D2.54mm_Drill1.5mm_Beaded
- TP13: value TestPoint -> TempHum SCL; footprint (none) -> TestPoint:TestPoint_Loop_D2.54mm_Drill1.5mm_Beaded
- TP7: value TestPoint -> Pot ADC; footprint (none) -> TestPoint:TestPoint_Loop_D2.54mm_Drill1.5mm_Beaded
- TP8: value TestPoint -> Therm ADC; footprint (none) -> TestPoint:TestPoint_Loop_D2.54mm_Drill1.5mm_Beaded
- TP9: value TestPoint -> Light SDA; footprint (none) -> TestPoint:TestPoint_Loop_D2.54mm_Drill1.5mm_Beaded
- U4: footprint (none) -> footprint:DFN-6_L2.0-W2.0-P0.50-BL-EP
- U5: footprint OptoDevice:Lite-On_LTR-303ALS-01 -> footprint:SOT-363_L2.0-W1.3-P0.65-LS2.1-BL
Changed lines of the file:
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@@
       (effects (font (size 1.27 1.27)) (justify left))
     )
-    (property "Value" "TestPoint" (at 191.77 37.465 90)
-      (effects (font (size 1.27 1.27)) (justify left))
-    )
-    (property "Footprint" "" (at 186.69 40.64 0)
+    (property "Value" "Light SCL" (at 191.77 37.465 90)
+      (effects (font (size 1.27 1.27)) (justify left))
+    )
+    (property "Footprint" "TestPoint:TestPoint_Loop_D2.54mm_Drill1.5mm_Beaded" (at 186.69 40.64 0)
       (effects (font (size 1.27 1.27)) hide)
     )
@@
       (effects (font (size 1.27 1.27)) (justify left))
     )
-    (property "Value" "TestPoint" (at 191.77 42.545 90)
-      (effects (font (size 1.27 1.27)) (justify left))
-    )
-    (property "Footprint" "" (at 186.69 45.72 0)
+    (property "Value" "Light Interrupt" (at 191.77 42.545 90)
+      (effects (font (size 1.27 1.27)) (justify left))
+    )
+    (property "Footprint" "TestPoint:TestPoint_Loop_D2.54mm_Drill1.5mm_Beaded" (at 186.69 45.72 0)
       (effects (font (size 1.27 1.27)) hide)
     )
@@
       (effects (font (size 1.27 1.27)) (justify left))
     )
-    (property "Value" "TestPoint" (at 191.77 32.385 90)
-      (effects (font (size 1.27 1.27)) (justify left))
-    )
-    (property "Footprint" "" (at 186.69 35.56 0)
+    (property "Value" "Light SDA" (at 191.77 32.385 90)
+      (effects (font (size 1.27 1.27)) (justify left))
+    )
+    (property "Footprint" "TestPoint:TestPoint_Loop_D2.54mm_Drill1.5mm_Beaded" (at 186.69 35.56 0)
       (effects (font (size 1.27 1.27)) hide)
     )
@@
       (effects (font (size 1.27 1.27)) (justify left))
     )
-    (property "Footprint" "Package_TO_SOT_SMD:SOT-23" (at 231.14 93.345 0)
+    (property "Footprint" "footprint:SOT-23_L2.9-W1.3-P1.90-LS2.4-BR" (at 231.14 93.345 0)
       (effects (font (size 1.27 1.27) italic) (justify left) hide)
     )
@@
       (effects (font (size 1.27 1.27)) (justify left))
     )
-    (property "Value" "TestPoint" (at 132.08 50.673 0)
-      (effects (font (size 1.27 1.27)) (justify left))
-    )
-    (property "Footprint" "" (at 134.62 52.07 0)
+    (property "Value" "Pot ADC" (at 132.08 50.673 0)
+      (effects (font (size 1.27 1.27)) (justify left))
+    )
+    (property "Footprint" "TestPoint:TestPoint_Loop_D2.54mm_Drill1.5mm_Beaded" (at 134.62 52.07 0)
       (effects (font (size 1.27 1.27)) hide)
     )
@@
       (effects (font (size 1.27 1.27)) (justify right))
     )
-    (property "Footprint" "" (at 236.728 29.21 90)
+    (property "Footprint" "footprint:R0603" (at 236.728 29.21 90)
       (effects (font (size 1.27 1.27)) hide)
     )
@@
       (effects (font (size 1.27 1.27)) (justify left))
     )
-    (property "Footprint" "Package_TO_SOT_SMD:SOT-23" (at 121.92 93.345 0)
+    (property "Footprint" "footprint:SOT-23_L2.9-W1.3-P1.90-LS2.4-BR" (at 121.92 93.345 0)
       (effects (font (size 1.27 1.27) italic) (justify left) hide)
     )
@@
       (effects (font (size 1.27 1.27)) (justify left))
     )
-    (property "Value" "TestPoint" (at 194.31 89.535 90)
-      (effects (font (size 1.27 1.27)) (justify left))
-    )
-    (property "Footprint" "" (at 189.23 92.71 0)
+    (property "Value" "TempHum SDA" (at 194.31 89.535 90)
+      (effects (font (size 1.27 1.27)) (justify left))
+    )
+    (property "Footprint" "TestPoint:TestPoint_Loop_D2.54mm_Drill1.5mm_Beaded" (at 189.23 92.71 0)
       (effects (font (size 1.27 1.27)) hide)
     )
@@
       (effects (font (size 1.27 1.27)) (justify right))
     )
-    (property "Footprint" "" (at 126.238 105.41 90)
+    (property "Footprint" "footprint:R1206" (at 126.238 105.41 90)
       (effects (font (size 1.27 1.27)) hide)
     )
@@
       (effects (font (size 1.27 1.27)) (justify right))
     )
-    (property "Footprint" "" (at 235.458 85.09 90)
+    (property "Footprint" "footprint:R0603" (at 235.458 85.09 90)
       (effects (font (size 1.27 1.27)) hide)
     )
@@
       (effects (font (size 1.27 1.27)) (justify right))
     )
-    (property "Footprint" "" (at 126.238 85.09 90)
+    (property "Footprint" "footprint:R0603" (at 126.238 85.09 90)
       (effects (font (size 1.27 1.27)) hide)
     )
@@
       (effects (font (size 1.27 1.27)) (justify left))
     )
-    (property "Footprint" "Package_TO_SOT_SMD:SOT-23" (at 232.41 37.465 0)
+    (property "Footprint" "footprint:SOT-23_L2.9-W1.3-P1.90-LS2.4-BR" (at 232.41 37.465 0)
       (effects (font (size 1.27 1.27) italic) (justify left) hide)
     )
@@
       (effects (font (size 1.27 1.27)) (justify left))
     )
-    (property "Value" "TestPoint" (at 137.16 106.553 0)
-      (effects (font (size 1.27 1.27)) (justify left))
-    )
-    (property "Footprint" "" (at 139.7 107.95 0)
+    (property "Value" "Therm ADC" (at 137.16 106.553 0)
+      (effects (font (size 1.27 1.27)) (justify left))
+    )
+    (property "Footprint" "TestPoint:TestPoint_Loop_D2.54mm_Drill1.5mm_Beaded" (at 139.7 107.95 0)
       (effects (font (size 1.27 1.27)) hide)
     )
@@
       (effects (font (size 1.27 1.27)) (justify left))
     )
-    (property "Value" "TestPoint" (at 194.31 94.615 90)
-      (effects (font (size 1.27 1.27)) (justify left))
-    )
-    (property "Footprint" "" (at 189.23 97.79 0)
+    (property "Value" "TempHum SCL" (at 194.31 94.615 90)
+      (effects (font (size 1.27 1.27)) (justify left))
+    )
+    (property "Footprint" "TestPoint:TestPoint_Loop_D2.54mm_Drill1.5mm_Beaded" (at 189.23 97.79 0)
       (effects (font (size 1.27 1.27)) hide)
     )
@@
       (effects (font (size 1.27 1.27)) (justify right))
     )
-    (property "Footprint" "" (at 218.948 90.17 90)
+    (property "Footprint" "footprint:R0603" (at 218.948 90.17 90)
       (effects (font (size 1.27 1.27)) hide)
     )
@@
       (effects (font (size 1.27 1.27)) (justify right))
     )
-    (property "Footprint" "" (at 220.218 34.29 90)
+    (property "Footprint" "footprint:R0603" (at 220.218 34.29 90)
       (effects (font (size 1.27 1.27)) hide)
     )
@@
       (effects (font (size 1.27 1.27)) (justify left))
     )
-    (property "Footprint" "" (at 202.8952 57.15 0)
+    (property "Footprint" "footprint:C0402" (at 202.8952 57.15 0)
       (effects (font (size 1.27 1.27)) hide)
     )
@@
       (effects (font (size 1.27 1.27)) (justify right))
     )
-    (property "Footprint" "" (at 109.728 90.17 90)
+    (property "Footprint" "footprint:R0603" (at 109.728 90.17 90)
       (effects (font (size 1.27 1.27)) hide)
     )
@@
       (effects (font (size 1.27 1.27)) (justify right))
     )
-    (property "Footprint" "" (at 124.46 54.61 0)
+    (property "Footprint" "footprint:RES-ADJ-TH_RK09K1130AJ3" (at 124.46 54.61 0)
       (effects (font (size 1.27 1.27)) hide)
     )
@@
       (effects (font (size 1.27 1.27)) (justify left))
     )
-    (property "Footprint" "" (at 185.1152 114.3 0)
+    (property "Footprint" "footprint:C0402_NEW" (at 185.1152 114.3 0)
       (effects (font (size 1.27 1.27)) hide)
     )
@@
       (effects (font (size 1.27 1.27)))
     )
-    (property "Footprint" "OptoDevice:Lite-On_LTR-303ALS-01" (at 234.95 44.45 0)
+    (property "Footprint" "footprint:SOT-363_L2.0-W1.3-P0.65-LS2.1-BL" (at 234.95 44.45 0)
       (effects (font (size 1.27 1.27)) hide)
     )
@@
       (effects (font (size 1.27 1.27)) (justify right))
     )
-    (property "Footprint" "" (at 126.238 34.29 90)
+    (property "Footprint" "footprint:R0603" (at 126.238 34.29 90)
       (effects (font (size 1.27 1.27)) hide)
     )
@@
       (effects (font (size 1.27 1.27)) (justify right))
     )
-    (property "Footprint" "" (at 109.728 39.37 90)
+    (property "Footprint" "footprint:R0603" (at 109.728 39.37 90)
       (effects (font (size 1.27 1.27)) hide)
     )
@@
       (effects (font (size 1.27 1.27)) (justify left))
     )
-    (property "Footprint" "Package_TO_SOT_SMD:SOT-23" (at 121.92 42.545 0)
+    (property "Footprint" "footprint:SOT-23_L2.9-W1.3-P1.90-LS2.4-BR" (at 121.92 42.545 0)
       (effects (font (size 1.27 1.27) italic) (justify left) hide)
     )
@@
       (effects (font (size 1.27 1.27)))
     )
-    (property "Footprint" "" (at 233.68 111.76 0)
+    (property "Footprint" "footprint:DFN-6_L2.0-W2.0-P0.50-BL-EP" (at 233.68 111.76 0)
       (effects (font (size 1.27 1.27)) hide)
     )
@@
       (effects (font (size 1.27 1.27)) (justify left))
     )
-    (property "Footprint" "" (at 124.46 115.57 0)
-      (effects (font (size 1.27 1.27)) hide)
-    )
+    (property "Footprint" "footprint:R0402" (at 124.46 115.57 0)
+      (effects (font (size 1.27 1.27)) hide)
+    )
