File: KiCad/power.kicad_sch (KiCad schematic)
At the start: 45 parts, among them J1 01x02_male_header, J2 01x02_male_header, Q1 AO3401A, Q2 AO3401A, Q3 AO3401A, Q4 AO3401A, U1 LMV321IDBVR, U2 Battery Charger, U4 XC6206PxxxMR, u3 battery holder

Commit message: Final schematic changes and start board design
Parts:
- C1, C2, C3, C4: footprint footprint:C0603 -> JLCPartFootprints:C0603
- D1: footprint footprint:SOD-123_L2.8-W1.8-LS3.7-RD -> JLCPartFootprints:SOD-123_L2.8-W1.8-LS3.7-RD
- D2, D3: footprint (none) -> JLCPartFootprints:LED0603-RD
- J1, J2: footprint footprint:HDR-TH_2P-P2.54-V-M -> Connector_PinHeader_2.54mm:PinHeader_1x02_P2.54mm_Vertical
- Q1, Q2, Q3, Q4: footprint footprint:SOT-23_L2.9-W1.3-P1.90-LS2.4-BR -> JLCPartFootprints:SOT-23_L2.9-W1.3-P1.90-LS2.4-BR
- R11: renamed from R12; footprint footprint:R0805 -> JLCPartFootprints:R0805
- R12: renamed from R13; footprint footprint:R0805 -> JLCPartFootprints:R0805
- R13: renamed from R14; footprint footprint:R0603 -> JLCPartFootprints:R0603
- R14: renamed from R15; footprint footprint:R0805 -> JLCPartFootprints:R0805
- R17: renamed from R18; footprint footprint:R0805 -> JLCPartFootprints:R0805
- R22: renamed from R23; footprint footprint:R0805 -> JLCPartFootprints:R0805
- R3: renamed from R4; footprint footprint:R0805 -> JLCPartFootprints:R0805
- R5: renamed from R6; footprint footprint:R0805 -> JLCPartFootprints:R0805
- R6: renamed from R7; footprint footprint:R0805 -> JLCPartFootprints:R0805
- R7: renamed from R8; footprint footprint:R0805 -> JLCPartFootprints:R0805
- R8: renamed from R9; footprint footprint:R0805 -> JLCPartFootprints:R0805
- R9: renamed from R10; footprint footprint:R0805 -> JLCPartFootprints:R0805
- R? (x11): footprint footprint:R0603 -> JLCPartFootprints:R0603
- TP? (x5): footprint footprint:Testpoint_2.54mm -> CustomFootprints:Testpoint; DNF (none) -> X
- U1: footprint footprint:SOT-23-5_L3.0-W1.7-P0.95-LS2.8-BR -> JLCPartFootprints:SOT-23-5_L3.0-W1.7-P0.95-LS2.8-BR
- U2: footprint footprint:ESOP-8_L4.9-W3.9-P1.27-LS6.0-BL-EP -> JLCPartFootprints:ESOP-8_L4.9-W3.9-P1.27-LS6.0-BL-EP
- U4: footprint footprint:SOT-23-3_L2.9-W1.6-P1.90-LS2.8-BR -> JLCPartFootprints:SOT-23-3_L2.9-W1.6-P1.90-LS2.8-BR
- u3: footprint footprint:BATTERY-SMD_18650-1S-L77.1-W20.7-1 -> JLCPartFootprints:BATTERY-SMD_18650-1S-L77.1-W20.7-1; DNF x -> X
