File: Temp/EEE3088F_CKR_backup.kicad_pcb (KiCad board)
At the start: 2 copper layers, 90 x 75 mm, 132 parts, among them J1 01x02_male_header, J2 01x02_male_header, J3 STM32F051C6_female_header, J4 STM32F051C6_testpoints, J5 STM-link_debugger, J6 01x10_male_header, Q1 AO3401A, Q2 AO3401A, Q3 AO3401A, Q4 AO3401A, Q5 AO3401A, Q6 AO3401A, Q7 AO3401A, Q8 AO3401A, SW1 Reset switch, SW2 Switch, SW3 Switch, SW4 Switch, U1 LMV321IDBVR, U2 Battery Charger, U4 XC6206PxxxMR, U5 GXHTC3, U6 LTR-303ALS-01, U7 24LC256, U8 usb, U9 HT42B534-2, Y1 Crystal

Commit message: made backup of PCB layout
Parts:
- renumbered B1 to u3
Connections:
- C2 pad 1: Net-(B1-+) -> Net-(J1-Pin_2)
- C5 pad 1: Net-(#FLG05-pwr) -> Net-(Q7-D)
- C6 pad 1: Net-(#FLG06-pwr) -> Net-(Q8-D)
- Q7 pad 3: Net-(#FLG05-pwr) -> Net-(Q7-D)
- Q8 pad 3: Net-(#FLG06-pwr) -> Net-(Q8-D)
- R15 pad 2: Net-(B1-+) -> Net-(J1-Pin_2)
- U2 pad 5: Net-(B1-+) -> Net-(J1-Pin_2)
- U5 pad 1: Net-(#FLG05-pwr) -> Net-(Q7-D)
- U6 pad 1: Net-(#FLG06-pwr) -> Net-(Q8-D)
