File: kian last changes/EEE3088F_CKR.kicad_pcb (KiCad board)
At the start: 2 copper layers, 90 x 75 mm, 131 parts, among them J1 01x02_male_header, J2 01x02_male_header, J3 STM32F051C6_female_header, J4 STM32F051C6_testpoints, J5 STM-link_debugger, J6 01x10_male_header, Q1 AO3401A, Q2 AO3400A, Q3 AO3401A, Q4 AO3401A, Q5 AO3401A, Q6 AO3401A, Q7 AO3401A, Q8 AO3401A, Q90 AO3401A, SW1 Reset switch, SW2 Switch, SW3 Switch, SW4 Switch, U1 LMS33460MG_NOPB, U2 Battery Charger, U4 XC6206PxxxMR, U5 GXHTC3, U6 LTR-303ALS-01, U7 24LC256, U8 usb, U9 HT42B534-2, Y1 Crystal

Commit message: made final production files
Connections:
- B1 pad 1: Net-(J1-Pin_2) -> Net-(B1-+)
- C5 pad 1: Net-(#FLG05-pwr) -> Net-(Q7-D)
- J1 pad 2: Net-(J1-Pin_2) -> Net-(B1-+)
- Q7 pad 3: Net-(#FLG05-pwr) -> Net-(Q7-D)
- R16 pad 2: Net-(J1-Pin_2) -> Net-(B1-+)
- R30 pad 1: Net-(Q8-D) -> Net-(#FLG06-pwr)
- TP3 pad 1: Net-(J1-Pin_2) -> Net-(B1-+)
- U5 pad 1: Net-(#FLG05-pwr) -> Net-(Q7-D)
Routing:
- net Net-(J1-Pin_2): track 83.1 -> 0.00 mm, vias 1 -> 0
- net Net-(B1-+): track 0.00 -> 83.1 mm, vias 0 -> 1
- net Net-(Q8-D): track 15.4 -> 0.00 mm
- net Net-(#FLG06-pwr): track 0.00 -> 15.4 mm
- net +3V3: track 256.6 -> 253.9 mm
- net /Microcontroller/NSRT: track 159.3 -> 160.2 mm
- net Net-(Q2-G): track 16.3 -> 17.1 mm
- net GND: vias 57 -> 58
Other:
- board text added: "R620"
- board text added: "Robert Dugmore - DGMROB001 Cameron Clark - CLRCAM007 Kian Frassek - FRSKIA001 EEE3088F 2023 Group 12 Sensor HAT PCB rev 0.3"
- board text removed: "Robert Dugmore - DGMROB001 Cameron Clark - CLRCAM007 Kian Frassek - FRSKIA001 EEE3088F 2023 Group 12 Sensor HAT PCB rev 0.2"
