File: kian last changes/USB.kicad_sch (KiCad schematic)
At the start: 11 parts, among them J6 01x10_male_header, U9 HT42B534-2

Commit message: residual changes
Parts:
- R1: JLCPCB Part # (none) -> C21189; JLCPSB Part # C21189 -> (none)
- R12: JLCPCB Part # (none) -> C4184; JLCPSB Part # C4184 -> (none)
- R12: JLCPCB Part # (none) -> C17414; JLCPSB Part # C17414 -> (none)
- U9: JLCPCB Part # (none) -> C493294; JLCPSB Part # C493294 -> (none)
- U?: JLCPCB Part # (none) -> C404969; JLCPSB Part # C404969 -> (none)
Changed lines of the file:
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@@
       (effects (font (size 1.27 1.27)) hide)
     )
-    (property "JLCPSB Part #" "C4184" (at 246.38 153.67 0)
+    (property "JLCPCB Part #" "C4184" (at 246.38 153.67 0)
       (effects (font (size 1.27 1.27)) hide)
     )
@@
       (effects (font (size 1.27 1.27)) hide)
     )
-    (property "JLCPSB Part #" "" (at 189.23 146.05 0)
+    (property "JLCPCB Part #" "" (at 189.23 146.05 0)
       (effects (font (size 1.27 1.27)) hide)
     )
@@
       (effects (font (size 1.27 1.27)) hide)
     )
-    (property "JLCPSB Part #" "" (at 186.69 102.87 0)
+    (property "JLCPCB Part #" "" (at 186.69 102.87 0)
       (effects (font (size 1.27 1.27)) hide)
     )
@@
       (effects (font (size 1.27 1.27)) hide)
     )
-    (property "JLCPSB Part #" "" (at 189.23 143.51 0)
+    (property "JLCPCB Part #" "" (at 189.23 143.51 0)
       (effects (font (size 1.27 1.27)) hide)
     )
@@
       (effects (font (size 1.27 1.27)) hide)
     )
-    (property "JLCPSB Part #" "" (at 255.27 114.3 0)
+    (property "JLCPCB Part #" "" (at 255.27 114.3 0)
       (effects (font (size 1.27 1.27)) hide)
     )
@@
       (effects (font (size 1.27 1.27)) hide)
     )
-    (property "JLCPSB Part #" "" (at 255.27 92.71 0)
+    (property "JLCPCB Part #" "" (at 255.27 92.71 0)
       (effects (font (size 1.27 1.27)) hide)
     )
@@
       (effects (font (size 1.27 1.27)) hide)
     )
-    (property "JLCPSB Part #" "C21189" (at 196.85 107.95 0)
+    (property "JLCPCB Part #" "C21189" (at 196.85 107.95 0)
       (effects (font (size 1.27 1.27)) hide)
     )
@@
       (effects (font (size 1.27 1.27)) hide)
     )
-    (property "JLCPSB Part #" "C493294" (at 214.63 142.24 0)
+    (property "JLCPCB Part #" "C493294" (at 214.63 142.24 0)
       (effects (font (size 1.27 1.27)) hide)
     )
@@
       (effects (font (size 1.27 1.27)) hide)
     )
-    (property "JLCPSB Part #" "C404969" (at 170.18 148.59 0)
+    (property "JLCPCB Part #" "C404969" (at 170.18 148.59 0)
       (effects (font (size 1.27 1.27)) hide)
     )
@@
       (effects (font (size 1.27 1.27)) hide)
     )
-    (property "JLCPSB Part #" "C17414" (at 246.38 143.51 0)
+    (property "JLCPCB Part #" "C17414" (at 246.38 143.51 0)
       (effects (font (size 1.27 1.27)) hide)
     )
@@
       (effects (font (size 1.27 1.27)) hide)
     )
-    (property "JLCPSB Part #" "C21189" (at 256.54 148.59 0)
-      (effects (font (size 1.27 1.27)) hide)
-    )
+    (property "JLCPCB Part #" "C21189" (at 256.54 148.59 0)
+      (effects (font (size 1.27 1.27)) hide)
+    )
