File: kian last changes/microcontroller.kicad_sch (KiCad schematic)
At the start: 52 parts, among them J3 STM32F051C6_female_header, J4 STM32F051C6_testpoints, J5 STM-link_debugger, SW1 Reset switch, SW2 Switch, SW3 Switch, SW4 Switch, U7 24LC256, Y1 Crystal

Commit message: residual changes
Parts:
- C7, C8: JLCPCB Part # (none) -> C1570; JLCPSB Part # C1570 -> (none)
- D4, D5: JLCPCB Part # (none) -> C34499; JLCPSB Part # C34499 -> (none)
- R33, R34, R35, R36, R37, R40, R41, R42, R43, R44, R45, R46, R47, R48, R55, R56, R57, R? (x2): JLCPCB Part # (none) -> C21189; JLCPSB Part # C21189 -> (none)
- R38, R39: JLCPCB Part # (none) -> C17630; JLCPSB Part # C17630 -> (none)
- R49: JLCPCB Part # (none) -> C17414; JLCPSB Part # C17414 -> (none)
- R? (x2): JLCPCB Part # (none) -> C51721; JLCPSB Part # C51721 -> (none)
- R?: JLCPCB Part # (none) -> C25924; JLCPSB Part # C25924 -> (none)
- SW1, SW2, SW3, SW4: JLCPCB Part # (none) -> C318884; JLCPSB Part # C318884 -> (none)
- U7: JLCPCB Part # (none) -> C411624; JLCPSB Part # C411624 -> (none)
- Y1: JLCPCB Part # (none) -> C12674; JLCPSB Part # C12674 -> (none)
