File: kian last changes/power.kicad_sch (KiCad schematic)
At the start: 46 parts, among them J1 01x02_male_header, J2 01x02_male_header, Q1 AO3401A, Q2 AO3400A, Q3 AO3401A, Q4 AO3401A, Q90 AO3401A, U1 LMS33460MG_NOPB, U2 Battery Charger, U4 XC6206PxxxMR

Commit message: residual changes
Parts:
- B1: JLCPCB Part # (none) -> C2988620; JLCPSB Part # C2988620 -> (none)
- C1, C2, C3, C4: JLCPCB Part # (none) -> C19702; JLCPSB Part # C19702 -> (none)
- D2: JLCPCB Part # (none) -> C72043; JLCPSB Part # C72043 -> (none)
- D3: JLCPCB Part # (none) -> C2286; JLCPSB Part # C2286 -> (none)
- Q1, Q3, Q4, Q90: JLCPCB Part # (none) -> C15127; JLCPSB Part # C15127 -> (none)
- Q2: JLCPCB Part # (none) -> C20917; JLCPSB Part # C20917 -> (none)
- R11, R14, R17, R22, R3, R9: JLCPCB Part # (none) -> C17630; JLCPSB Part # C17630 -> (none)
- R? (x14): JLCPCB Part # (none) -> C21189; JLCPSB Part # C21189 -> (none)
- R?: JLCPCB Part # (none) -> C4184; JLCPSB Part # C4184 -> (none)
- R? (x2): JLCPCB Part # (none) -> C149504; JLCPSB Part # C149504 -> (none)
- R?: JLCPCB Part # (none) -> C17709; JLCPSB Part # C17709 -> (none)
- U1: JLCPCB Part # (none) -> C95686; JLCPSB Part # C95686 -> (none)
- U2: JLCPCB Part # (none) -> C16581; JLCPSB Part # C16581 -> (none)
- U4: JLCPCB Part # (none) -> C5446; JLCPSB Part # C5446 -> (none)
