File: kian last changes/sensors.kicad_sch (KiCad schematic)
At the start: 24 parts, among them U5 GXHTC3, U6 LTR-303ALS-01

Commit message: residual changes
Parts:
- C?: JLCPCB Part # (none) -> C52923; JLCPSB Part # C52923 -> (none)
- C?: JLCPCB Part # (none) -> C1525; JLCPSB Part # C1525 -> (none)
- Q? (x4): JLCPCB Part # (none) -> C15127; JLCPSB Part # C15127 -> (none)
- R? (x8): JLCPCB Part # (none) -> C21189; JLCPSB Part # C21189 -> (none)
- R?: JLCPCB Part # (none) -> C17900; JLCPSB Part # C17900 -> (none)
- RV1: JLCPCB Part # (none) -> C388854; JLCPSB Part # C388854 -> (none)
- TH1: JLCPCB Part # (none) -> C77130; JLCPSB Part # C77130 -> (none)
- U5: JLCPCB Part # (none) -> C2837688; JLCPSB Part # C2837688 -> (none)
- U6: JLCPCB Part # (none) -> C364577; JLCPSB Part # C364577 -> (none)
Changed lines of the file:
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@@
       (effects (font (size 1.27 1.27)) hide)
     )
-    (property "JLCPSB Part #" "" (at 133.35 149.86 0)
+    (property "JLCPCB Part #" "" (at 133.35 149.86 0)
       (effects (font (size 1.27 1.27)) hide)
     )
@@
       (effects (font (size 1.27 1.27)) hide)
     )
-    (property "JLCPSB Part #" "" (at 186.69 40.64 0)
+    (property "JLCPCB Part #" "" (at 186.69 40.64 0)
       (effects (font (size 1.27 1.27)) hide)
     )
@@
       (effects (font (size 1.27 1.27)) hide)
     )
-    (property "JLCPSB Part #" "" (at 133.35 137.16 0)
+    (property "JLCPCB Part #" "" (at 133.35 137.16 0)
       (effects (font (size 1.27 1.27)) hide)
     )
@@
       (effects (font (size 1.27 1.27)) hide)
     )
-    (property "JLCPSB Part #" "C15127" (at 236.22 95.25 0)
+    (property "JLCPCB Part #" "C15127" (at 236.22 95.25 0)
       (effects (font (size 1.27 1.27)) hide)
     )
@@
       (effects (font (size 1.27 1.27)) hide)
     )
-    (property "JLCPSB Part #" "" (at 129.54 52.07 0)
+    (property "JLCPCB Part #" "" (at 129.54 52.07 0)
       (effects (font (size 1.27 1.27)) hide)
     )
@@
       (effects (font (size 1.27 1.27)) hide)
     )
-    (property "JLCPSB Part #" "C21189" (at 234.95 29.21 0)
+    (property "JLCPCB Part #" "C21189" (at 234.95 29.21 0)
       (effects (font (size 1.27 1.27)) hide)
     )
@@
       (effects (font (size 1.27 1.27)) hide)
     )
-    (property "JLCPSB Part #" "C15127" (at 127 95.25 0)
+    (property "JLCPCB Part #" "C15127" (at 127 95.25 0)
       (effects (font (size 1.27 1.27)) hide)
     )
@@
       (effects (font (size 1.27 1.27)) hide)
     )
-    (property "JLCPSB Part #" "C17900" (at 124.46 105.41 0)
+    (property "JLCPCB Part #" "C17900" (at 124.46 105.41 0)
       (effects (font (size 1.27 1.27)) hide)
     )
@@
       (effects (font (size 1.27 1.27)) hide)
     )
-    (property "JLCPSB Part #" "C21189" (at 233.68 85.09 0)
+    (property "JLCPCB Part #" "C21189" (at 233.68 85.09 0)
       (effects (font (size 1.27 1.27)) hide)
     )
@@
       (effects (font (size 1.27 1.27)) hide)
     )
-    (property "JLCPSB Part #" "C21189" (at 124.46 85.09 0)
+    (property "JLCPCB Part #" "C21189" (at 124.46 85.09 0)
       (effects (font (size 1.27 1.27)) hide)
     )
@@
       (effects (font (size 1.27 1.27)) hide)
     )
-    (property "JLCPSB Part #" "C15127" (at 237.49 39.37 0)
+    (property "JLCPCB Part #" "C15127" (at 237.49 39.37 0)
       (effects (font (size 1.27 1.27)) hide)
     )
@@
       (effects (font (size 1.27 1.27)) hide)
     )
-    (property "JLCPSB Part #" "" (at 134.62 107.95 0)
+    (property "JLCPCB Part #" "" (at 134.62 107.95 0)
       (effects (font (size 1.27 1.27)) hide)
     )
@@
       (effects (font (size 1.27 1.27)) hide)
     )
-    (property "JLCPSB Part #" "C21189" (at 217.17 90.17 0)
+    (property "JLCPCB Part #" "C21189" (at 217.17 90.17 0)
       (effects (font (size 1.27 1.27)) hide)
     )
@@
       (effects (font (size 1.27 1.27)) hide)
     )
-    (property "JLCPSB Part #" "C21189" (at 218.44 34.29 0)
+    (property "JLCPCB Part #" "C21189" (at 218.44 34.29 0)
       (effects (font (size 1.27 1.27)) hide)
     )
@@
       (effects (font (size 1.27 1.27)) hide)
     )
-    (property "JLCPSB Part #" "C52923" (at 201.93 53.34 0)
+    (property "JLCPCB Part #" "C52923" (at 201.93 53.34 0)
       (effects (font (size 1.27 1.27)) hide)
     )
@@
       (effects (font (size 1.27 1.27)) hide)
     )
-    (property "JLCPSB Part #" "C21189" (at 107.95 90.17 0)
+    (property "JLCPCB Part #" "C21189" (at 107.95 90.17 0)
       (effects (font (size 1.27 1.27)) hide)
     )
@@
       (effects (font (size 1.27 1.27)) hide)
     )
-    (property "JLCPSB Part #" "C388854" (at 124.46 54.61 0)
+    (property "JLCPCB Part #" "C388854" (at 124.46 54.61 0)
       (effects (font (size 1.27 1.27)) hide)
     )
@@
       (effects (font (size 1.27 1.27)) hide)
     )
-    (property "JLCPSB Part #" "C1525" (at 184.15 110.49 0)
+    (property "JLCPCB Part #" "C1525" (at 184.15 110.49 0)
       (effects (font (size 1.27 1.27)) hide)
     )
@@
       (effects (font (size 1.27 1.27)) hide)
     )
-    (property "JLCPSB Part #" "C364577" (at 234.95 55.88 0)
+    (property "JLCPCB Part #" "C364577" (at 234.95 55.88 0)
       (effects (font (size 1.27 1.27)) hide)
     )
@@
       (effects (font (size 1.27 1.27)) hide)
     )
-    (property "JLCPSB Part #" "C21189" (at 124.46 34.29 0)
+    (property "JLCPCB Part #" "C21189" (at 124.46 34.29 0)
       (effects (font (size 1.27 1.27)) hide)
     )
@@
       (effects (font (size 1.27 1.27)) hide)
     )
-    (property "JLCPSB Part #" "C21189" (at 107.95 39.37 0)
+    (property "JLCPCB Part #" "C21189" (at 107.95 39.37 0)
       (effects (font (size 1.27 1.27)) hide)
     )
@@
       (effects (font (size 1.27 1.27)) hide)
     )
-    (property "JLCPSB Part #" "C15127" (at 127 44.45 0)
+    (property "JLCPCB Part #" "C15127" (at 127 44.45 0)
       (effects (font (size 1.27 1.27)) hide)
     )
@@
       (effects (font (size 1.27 1.27)) hide)
     )
-    (property "JLCPSB Part #" "C2837688" (at 233.68 111.76 0)
+    (property "JLCPCB Part #" "C2837688" (at 233.68 111.76 0)
       (effects (font (size 1.27 1.27)) hide)
     )
@@
       (effects (font (size 1.27 1.27)) hide)
     )
-    (property "JLCPSB Part #" "C77130" (at 124.46 115.57 0)
-      (effects (font (size 1.27 1.27)) hide)
-    )
+    (property "JLCPCB Part #" "C77130" (at 124.46 115.57 0)
+      (effects (font (size 1.27 1.27)) hide)
+    )
